File: AlimentacionYCargador.kicad_sch (KiCad schematic)
At the start: 23 parts, among them Q1 2N7002, Q2 2N7002, Q3 2N7002, U2 BQ24075RGTR, U3 MCP1826S-3302E/DB

Commit message: Avance de sch
Parts:
- removed JP1: SolderJumper, Jumper:SolderJumper-2_P1.3mm_Open_RoundedPad1.0x1.5mm, symbol Jumper:SolderJumper_2_Open
- removed Q1, Q2, Q3: 2N7002, Package_TO_SOT_SMD:SOT-23, symbol Transistor_FET:2N7002
- removed R4, R8: 10K, Resistor_SMD:R_0402_1005Metric, symbol Device:R_Small
- removed TP2: TP, TestPoint:TestPoint_Pad_D2.5mm, symbol Connector:TestPoint
Connections:
- net SYSOFF is gone; now on net GND: U2.15 (SYSOFF)
Other:
- note removed: "PULL DOWN GATE EN SCH PRINCIPAL"

Commit message: listo para fabricar
Parts:
- C1, C4, C6: JLCPCB Part # (none) -> C1525
- C2, C5, C7: JLCPCB Part # (none) -> C45783
- C3: JLCPCB Part # (none) -> C52923
- FB1: JLCPCB Part # (none) -> C1017
- R4: renamed from R5; JLCPCB Part # (none) -> C25862
- R5: renamed from R6; JLCPCB Part # (none) -> C25862
- R6: renamed from R7; JLCPCB Part # (none) -> C25862
- R7: renamed from R9; JLCPCB Part # (none) -> C25744
- R8: renamed from R10; JLCPCB Part # (none) -> C25744
- R9: renamed from R11; JLCPCB Part # (none) -> C25744
- U2: JLCPCB Part # (none) -> C15464
- U3: JLCPCB Part # (none) -> C638624
Changed lines of the file:
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@@
+			)
+		)
+		(property "JLCPCB Part #" "C638624"
+			(at 143.51 48.26 0)
+			(effects
+				(font
+					(size 1.27 1.27)
+				)
+				(hide yes)
 			)
 		)
@@
 		(on_board yes)
 		(dnp no)
-		(property "Reference" "R10"
+		(property "Reference" "R8"
 			(at 116.078 75.184 0)
 			(effects
@@
 			)
 		)
+		(property "JLCPCB Part #" "C25744"
+			(at 118.11 74.93 0)
+			(effects
+				(font
+					(size 1.27 1.27)
+				)
+				(hide yes)
+			)
+		)
 		(pin "1"
 		)
@@
 			(project "ContadorPortatil"
 				(path "/49f8911c-9183-413a-8434-23c6add05009/bd1acdec-87a6-4a80-b9e7-38ccff3b632e"
-					(reference "R10")
+					(reference "R8")
 					(unit 1)
 				)
@@
 		(on_board yes)
 		(dnp no)
-		(property "Reference" "R9"
+		(property "Reference" "R7"
 			(at 99.568 62.738 90)
 			(effects
@@
 			)
 		)
+		(property "JLCPCB Part #" "C25744"
+			(at 97.79 60.96 90)
+			(effects
+				(font
+					(size 1.27 1.27)
+				)
+				(hide yes)
+			)
+		)
 		(pin "1"
 		)
@@
 			(project "ContadorPortatil"
 				(path "/49f8911c-9183-413a-8434-23c6add05009/bd1acdec-87a6-4a80-b9e7-38ccff3b632e"
-					(reference "R9")
+					(reference "R7")
 					(unit 1)
 				)
@@
 			)
 		)
+		(property "JLCPCB Part #" "C52923"
+			(at 111.76 53.34 0)
+			(effects
+				(font
+					(size 1.27 1.27)
+				)
+				(hide yes)
+			)
+		)
 		(pin "1"
 		)
@@
 			)
 		)
+		(property "JLCPCB Part #" "C45783"
+			(at 162.56 53.34 0)
+			(effects
+				(font
+					(size 1.27 1.27)
+				)
+				(hide yes)
+			)
+		)
 		(pin "1"
 		)
@@
 			)
 		)
+		(property "JLCPCB Part #" "C45783"
+			(at 59.69 39.37 0)
+			(effects
+				(font
+					(size 1.27 1.27)
+				)
+				(hide yes)
+			)
+		)
 		(pin "1"
 		)
@@
 		(on_board yes)
 		(dnp no)
-		(property "Reference" "R11"
+		(property "Reference" "R9"
 			(at 123.952 75.184 0)
 			(effects
@@
 			)
 		)
+		(property "JLCPCB Part #" "C25744"
+			(at 121.92 74.93 0)
+			(effects
+				(font
+					(size 1.27 1.27)
+				)
+				(hide yes)
+			)
+		)
 		(pin "1"
 		)
@@
 			(project "ContadorPortatil"
 				(path "/49f8911c-9183-413a-8434-23c6add05009/bd1acdec-87a6-4a80-b9e7-38ccff3b632e"
-					(reference "R11")
+					(reference "R9")
 					(unit 1)
 				)
@@
 		(on_board yes)
 		(dnp no)
-		(property "Reference" "R6"
+		(property "Reference" "R5"
 			(at 57.658 73.152 0)
 			(effects
@@
 			)
 		)
+		(property "JLCPCB Part #" "C25862"
+			(at 59.69 72.39 0)
+			(effects
+				(font
+					(size 1.27 1.27)
+				)
+				(hide yes)
+			)
+		)
 		(pin "1"
 		)
@@
 			(project "ContadorPortatil"
 				(path "/49f8911c-9183-413a-8434-23c6add05009/bd1acdec-87a6-4a80-b9e7-38ccff3b632e"
-					(reference "R6")
+					(reference "R5")
 					(unit 1)
 				)
@@
 			)
 		)
+		(property "JLCPCB Part #" "C1525"
+			(at 54.61 39.37 0)
+			(effects
+				(font
+					(size 1.27 1.27)
+				)
+				(hide yes)
+			)
+		)
 		(pin "1"
 		)
@@
 		(on_board yes)
 		(dnp no)
-		(property "Reference" "R5"
+		(property "Reference" "R4"
 			(at 52.578 60.452 0)
 			(effects
@@
 			)
 		)
+		(property "JLCPCB Part #" "C25862"
+			(at 54.61 59.69 0)
+			(effects
+				(font
+					(size 1.27 1.27)
+				)
+				(hide yes)
+			)
+		)
 		(pin "1"
 		)
@@
 			(project "ContadorPortatil"
 				(path "/49f8911c-9183-413a-8434-23c6add05009/bd1acdec-87a6-4a80-b9e7-38ccff3b632e"
-					(reference "R5")
+					(reference "R4")
 					(unit 1)
 				)
@@
 			)
 		)
+		(property "JLCPCB Part #" "C1525"
+			(at 157.48 53.34 0)
+			(effects
+				(font
+					(size 1.27 1.27)
+				)
+				(hide yes)
+			)
+		)
 		(pin "1"
 		)
@@
 			)
 		)
+		(property "JLCPCB Part #" "C1017"
+			(at 118.11 48.26 90)
+			(effects
+				(font
+					(size 1.27 1.27)
+				)
+				(hide yes)
+			)
+		)
 		(pin "1"
 		)
@@
 		)
 		(property "Sim.Pins" ""
+			(at 129.54 53.34 0)
+			(effects
+				(font
+					(size 1.27 1.27)
+				)
+				(hide yes)
+			)
+		)
+		(property "JLCPCB Part #" "C45783"
 			(at 129.54 53.34 0)
 			(effects
@@
 			)
 		)
+		(property "JLCPCB Part #" "C15464"
+			(at 82.55 58.42 0)
+			(effects
+				(font
+					(size 1.27 1.27)
+				)
+				(hide yes)
+			)
+		)
 		(pin "11"
 		)
@@
 			)
 		)
+		(property "JLCPCB Part #" "C1525"
+			(at 124.46 53.34 0)
+			(effects
+				(font
+					(size 1.27 1.27)
+				)
+				(hide yes)
+			)
+		)
 		(pin "1"
 		)
@@
 		(on_board yes)
 		(dnp no)
-		(property "Reference" "R7"
+		(property "Reference" "R6"
 			(at 64.262 73.152 0)
 			(effects
@@
 			)
 		)
+		(property "JLCPCB Part #" "C25862"
+			(at 62.23 72.39 0)
+			(effects
+				(font
+					(size 1.27 1.27)
+				)
+				(hide yes)
+			)
+		)
 		(pin "1"
 		)
@@
 			(project "ContadorPortatil"
 				(path "/49f8911c-9183-413a-8434-23c6add05009/bd1acdec-87a6-4a80-b9e7-38ccff3b632e"
-					(reference "R7")
-					(unit 1)
-				)
+					(reference "R6")
+					(unit 1)
+				)
