File: ESP32-Portatil.kicad_sch (KiCad schematic)
At the start: 9 parts, among them J1 GT-USB-7047A, SW1 SW_SPST, U1 DM-OLED096-636

Commit message: Avance de sch
Parts:
- removed R3: 10K, Resistor_SMD:R_0402_1005Metric, symbol Device:R_Small
- removed SW1: SW_SPST, Button_Switch_THT:SW_PUSH_6mm, symbol Switch:SW_SPST
- removed TP1: TP, TestPoint:TestPoint_Pad_D2.5mm, symbol Connector:TestPoint
- added J2: TM-2027, TNG_Connectors:TM-2027, symbol TNG_Connectors:TM-2027
- added J3: SLLB510100, TNG_Connectors:SLLB510100, symbol TNG_Connectors:SLLB510100
Connections:
- no-connect marks 3 -> 2
Other:
- sheet Alimentacion y cargador ports: added none; removed PULSADOR, PWR_ON_MCU, SYSOFF
- sheet MCU ports: added none; removed PWR_ON

Commit message: Casi que placa lista
Parts:
- added Q1: AO3401A, Package_TO_SOT_SMD:SOT-23, symbol Transistor_FET:AO3401A
- added R8: 10K, Resistor_SMD:R_0402_1005Metric, symbol Device:R_Small
Connections:
- net +3V3: now also Q1.2 (S), R8.1; no longer U1.2 (VCC_IN)
- net GND: now also J2.4 (Com), J3.C
- net SW_ROT_1: now reaches J3.1
- net SW_ROT_2: now reaches J3.2
- net SW_ROT_T: now reaches J3.T
- net SW_MULT_A: now reaches J2.1 (A)
- net SW_MULT_B: now reaches J2.2 (B)
- net SW_MULT_C: now reaches J2.3 (C)
- net SW_MULT_D: now reaches J2.5 (D)
- net SW_MULT_pul: now reaches J2.6 (Cen)
- new net: Q1.3 (D), U1.2 (VCC_IN)
- new net DISP_ON: Q1.1 (G), R8.2
Other:
- sheet MCU ports: added DISP_ON, SW_MUL_DW, SW_MUL_L, SW_MUL_R, SW_MUL_UP, SW_MUL_pul, SW_ROT_CCW, SW_ROT_CW, SW_ROT_T, VBAT; removed PULSADOR, PULSE_IN
- moved on the sheet: J2, J3, U1

Commit message: listo para fabricar
Parts:
- H1, H2, U1: JLCPCB Part # (none) -> -
- J1: JLCPCB Part # (none) -> C963216
- Q1: JLCPCB Part # (none) -> C15127
- R1, R2: JLCPCB Part # (none) -> C25905
- R3: renamed from R8; JLCPCB Part # (none) -> C25744
Changed lines of the file:
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@@
+			)
+		)
+		(property "JLCPCB Part #" "-"
+			(at 187.96 22.86 0)
+			(effects
+				(font
+					(size 1.27 1.27)
+				)
+				(hide yes)
 			)
 		)
@@
 			)
 		)
+		(property "JLCPCB Part #" "-"
+			(at 177.8 22.86 0)
+			(effects
+				(font
+					(size 1.27 1.27)
+				)
+				(hide yes)
+			)
+		)
 		(pin "1"
 		)
@@
 		(dnp no)
 		(fields_autoplaced yes)
-		(property "Reference" "#PWR011"
+		(property "Reference" "#PWR012"
 			(at 175.26 53.34 0)
 			(effects
@@
 			(project "ESP32-Portatil"
 				(path "/49f8911c-9183-413a-8434-23c6add05009"
-					(reference "#PWR011")
+					(reference "#PWR012")
 					(unit 1)
 				)
@@
 		)
 		(property "Sim.Pins" ""
+			(at 58.42 35.56 90)
+			(effects
+				(font
+					(size 1.27 1.27)
+				)
+				(hide yes)
+			)
+		)
+		(property "JLCPCB Part #" "C25905"
 			(at 58.42 35.56 90)
 			(effects
@@
 			)
 		)
+		(property "JLCPCB Part #" "-"
+			(at 138.43 93.98 0)
+			(effects
+				(font
+					(size 1.27 1.27)
+				)
+				(hide yes)
+			)
+		)
 		(pin "2"
 		)
@@
 		(dnp no)
 		(fields_autoplaced yes)
-		(property "Reference" "#PWR012"
+		(property "Reference" "#PWR013"
 			(at 184.15 99.06 0)
 			(effects
@@
 			(project "ESP32-Portatil"
 				(path "/49f8911c-9183-413a-8434-23c6add05009"
-					(reference "#PWR012")
+					(reference "#PWR013")
 					(unit 1)
 				)
@@
 		(on_board yes)
 		(dnp no)
-		(property "Reference" "R8"
+		(property "Reference" "R3"
 			(at 107.188 95.758 90)
 			(effects
@@
 			)
 		)
+		(property "JLCPCB Part #" "C25744"
+			(at 105.41 93.98 90)
+			(effects
+				(font
+					(size 1.27 1.27)
+				)
+				(hide yes)
+			)
+		)
 		(pin "1"
 		)
@@
 			(project "ESP32-Portatil"
 				(path "/49f8911c-9183-413a-8434-23c6add05009"
-					(reference "R8")
+					(reference "R3")
 					(unit 1)
 				)
@@
 			)
 		)
+		(property "JLCPCB Part #" "C25905"
+			(at 58.42 33.02 90)
+			(effects
+				(font
+					(size 1.27 1.27)
+				)
+				(hide yes)
+			)
+		)
 		(pin "1"
 		)
@@
 		(dnp no)
 		(fields_autoplaced yes)
-		(property "Reference" "#PWR013"
+		(property "Reference" "#PWR011"
 			(at 177.8 31.75 0)
 			(effects
@@
 			(project "ContadorPortatil"
 				(path "/49f8911c-9183-413a-8434-23c6add05009"
-					(reference "#PWR013")
+					(reference "#PWR011")
 					(unit 1)
 				)
@@
 			)
 		)
+		(property "JLCPCB Part #" "C963216"
+			(at 31.75 43.18 0)
+			(effects
+				(font
+					(size 1.27 1.27)
+				)
+				(hide yes)
+			)
+		)
 		(pin "A8"
 		)
@@
 			(effects
 				(font
+					(size 1.27 1.27)
+				)
+				(hide yes)
+			)
+		)
+		(property "JLCPCB Part #" "C15127"
+			(at 113.03 88.9 90)
+			(effects
+				(font
