File: packBateria.kicad_sch (KiCad schematic)
At the start: 6 parts, among them Q4 IRF7341TRPBF, U4 BQ29700DSER

Commit message: Casi que placa lista
Parts:
- added TP4: BAT+, TestPoint:TestPoint_Loop_D1.80mm_Drill1.0mm_Beaded, symbol Connector:TestPoint
Connections:
- net B+: now also TP4.1
Changed lines of the file:
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@@
+	)
+	(junction
+		(at 116.84 45.72)
+		(diameter 0)
+		(color 0 0 0 0)
 	)
 	(junction
@@
 	(wire
 		(pts
-			(xy 111.76 45.72) (xy 119.38 45.72)
+			(xy 111.76 45.72) (xy 116.84 45.72)
 		)
 		(stroke
@@
 	(wire
 		(pts
+			(xy 116.84 45.72) (xy 119.38 45.72)
+		)
+		(stroke
+			(width 0)
+			(type default)
+		)
+	)
+	(wire
+		(pts
 			(xy 96.52 78.74) (xy 111.76 78.74)
 		)
@@
 		(pts
 			(xy 60.96 78.74) (xy 64.77 78.74)
+		)
+		(stroke
+			(width 0)
+			(type default)
+		)
+	)
+	(wire
+		(pts
+			(xy 116.84 38.1) (xy 116.84 45.72)
 		)
 		(stroke
@@
 					(unit 1)
 				)
+			)
+		)
+	)
+	(symbol
+		(lib_id "Connector:TestPoint")
+		(at 116.84 38.1 0)
+		(unit 1)
+		(exclude_from_sim no)
+		(in_bom yes)
+		(on_board yes)
+		(dnp no)
+		(fields_autoplaced yes)
+		(property "Reference" "TP4"
+			(at 119.38 33.5279 0)
+			(effects
+				(font
+					(size 1.27 1.27)
+				)
+				(justify left)
+			)
+		)
+		(property "Value" "BAT+"
+			(at 119.38 36.0679 0)
+			(effects
+				(font
+					(size 1.27 1.27)
+				)
+				(justify left)
+			)
+		)
+		(property "Footprint" "TestPoint:TestPoint_Loop_D1.80mm_Drill1.0mm_Beaded"
+			(at 121.92 38.1 0)
+			(effects
+				(font
+					(size 1.27 1.27)
+				)
+				(hide yes)
+			)
+		)
+		(property "Datasheet" "~"
+			(at 121.92 38.1 0)
+			(effects
+				(font
+					(size 1.27 1.27)
+				)
+				(hide yes)
+			)
+		)
+		(property "Description" "test point"
+			(at 116.84 38.1 0)
+			(effects
+				(font
+					(size 1.27 1.27)
+				)
+				(hide yes)
+			)
+		)
+		(pin "1"
+		)
+		(instances
+			(project ""
+				(path "/49f8911c-9183-413a-8434-23c6add05009/c80999d4-c78c-44aa-8cf7-da02a279d4f3"
+					(reference "TP4")
+					(unit 1)
+				)

Commit message: listo para fabricar
Parts:
- BT1: JLCPCB Part # (none) -> -
- C8: JLCPCB Part # (none) -> C1525
- Q2: renamed from Q4; JLCPCB Part # (none) -> C21791
- R10: renamed from R12; JLCPCB Part # (none) -> C25879
- R11: renamed from R13; JLCPCB Part # (none) -> C23138
- TP1: renamed from TP4; JLCPCB Part # (none) -> -
- U4: JLCPCB Part # (none) -> C183096
Changed lines of the file:
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@@
 		(on_board yes)
 		(dnp no)
-		(property "Reference" "Q4"
+		(property "Reference" "Q2"
 			(at 71.12 82.55 90)
 			(effects
@@
 		)
 		(property "Sim.Pins" ""
+			(at 71.12 76.2 90)
+			(effects
+				(font
+					(size 1.27 1.27)
+				)
+				(hide yes)
+			)
+		)
+		(property "JLCPCB Part #" "C21791"
 			(at 71.12 76.2 90)
 			(effects
@@
 			(project ""
 				(path "/49f8911c-9183-413a-8434-23c6add05009/c80999d4-c78c-44aa-8cf7-da02a279d4f3"
-					(reference "Q4")
+					(reference "Q2")
 					(unit 1)
 				)
@@
 			)
 		)
+		(property "JLCPCB Part #" "C1525"
+			(at 111.76 69.85 0)
+			(effects
+				(font
+					(size 1.27 1.27)
+				)
+				(hide yes)
+			)
+		)
 		(pin "1"
 		)
@@
 		(on_board yes)
 		(dnp no)
-		(property "Reference" "R12"
+		(property "Reference" "R10"
 			(at 62.23 63.4999 0)
 			(effects
@@
 		)
 		(property "Sim.Pins" ""
+			(at 64.77 64.77 0)
+			(effects
+				(font
+					(size 1.27 1.27)
+				)
+				(hide yes)
+			)
+		)
+		(property "JLCPCB Part #" "C25879"
 			(at 64.77 64.77 0)
 			(effects
@@
 			(project "ContadorPortatil"
 				(path "/49f8911c-9183-413a-8434-23c6add05009/c80999d4-c78c-44aa-8cf7-da02a279d4f3"
-					(reference "R12")
+					(reference "R10")
 					(unit 1)
 				)
@@
 		(on_board yes)
 		(dnp no)
-		(property "Reference" "R13"
+		(property "Reference" "R11"
 			(at 114.3 50.7999 0)
 			(effects
@@
 		)
 		(property "Sim.Pins" ""
+			(at 111.76 52.07 0)
+			(effects
+				(font
+					(size 1.27 1.27)
+				)
+				(hide yes)
+			)
+		)
+		(property "JLCPCB Part #" "C23138"
 			(at 111.76 52.07 0)
 			(effects
@@
 			(project ""
 				(path "/49f8911c-9183-413a-8434-23c6add05009/c80999d4-c78c-44aa-8cf7-da02a279d4f3"
-					(reference "R13")
+					(reference "R11")
 					(unit 1)
 				)
@@
 		(dnp no)
 		(fields_autoplaced yes)
-		(property "Reference" "TP4"
+		(property "Reference" "TP1"
 			(at 119.38 33.5279 0)
 			(effects
@@
 		)
 		(property "Description" "test point"
+			(at 116.84 38.1 0)
+			(effects
+				(font
+					(size 1.27 1.27)
+				)
+				(hide yes)
+			)
+		)
+		(property "JLCPCB Part #" "-"
 			(at 116.84 38.1 0)
 			(effects
@@
 			(project ""
 				(path "/49f8911c-9183-413a-8434-23c6add05009/c80999d4-c78c-44aa-8cf7-da02a279d4f3"
-					(reference "TP4")
+					(reference "TP1")
 					(unit 1)
 				)
@@
 			)
 		)
+		(property "JLCPCB Part #" "C183096"
+			(at 96.52 59.69 0)
+			(effects
+				(font
+					(size 1.27 1.27)
+				)
+				(hide yes)
+			)
+		)
 		(pin "5"
 		)
@@
 		(on_board yes)
 		(dnp no)
-		(property "Reference" "Q4"
+		(property "Reference" "Q2"
 			(at 81.28 82.55 90)
 			(effects
@@
 		)
 		(property "Sim.Pins" ""
+			(at 81.28 76.2 90)
+			(effects
+				(font
+					(size 1.27 1.27)
+				)
+				(hide yes)
+			)
+		)
+		(property "JLCPCB Part #" "C21791"
 			(at 81.28 76.2 90)
 			(effects
@@
 			(project ""
 				(path "/49f8911c-9183-413a-8434-23c6add05009/c80999d4-c78c-44aa-8cf7-da02a279d4f3"
-					(reference "Q4")
+					(reference "Q2")
 					(unit 2)
 				)
@@
 			(at 119.38 63.5 0)
 			(effects
+				(font
+					(size 1.27 1.27)
+				)
+				(hide yes)
+			)
+		)
+		(property "JLCPCB Part #" "-"
+			(at 119.38 63.5 0)
+			(effects
