File: ESP32-Portatil.kicad_pcb (KiCad board)
At the start: 4 copper layers, 26 x 109 mm, 46 parts, among them J1 GT-USB-7047A, Q1 2N7002, Q2 2N7002, Q3 2N7002, Q4 IRF7341TRPBF, Q5 2N7002, SW1 SW_SPST, U1 DM-OLED096-636, U2 BQ24075RGTR, U3 MCP1826S-3302E/DB, U4 BQ29700DSER, U6 ESP32-C6-MINI-1

Commit message: Avance de sch
Parts:
- removed JP1: SolderJumper, Jumper:SolderJumper-2_P1.3mm_Open_RoundedPad1.0x1.5mm
- removed Q1, Q2, Q3, Q5: 2N7002, Package_TO_SOT_SMD:SOT-23
- removed R19, R3, R4, R8: 10K, Resistor_SMD:R_0402_1005Metric
- removed SW1: SW_SPST, Button_Switch_THT:SW_PUSH_6mm
- removed TP1, TP2: TP, TestPoint:TestPoint_Pad_D2.5mm
- added C9: 100nF, Capacitor_SMD:C_0402_1005Metric, F.Cu at (160.0, 116.2)
- added J2: TM-2027, TNG_Connectors:TM-2027, F.Cu at (139.0, 94.0)
- added J3: SLLB510100, TNG_Connectors:SLLB510100, F.Cu at (148.5, 94.0)
- added U5: ADXL343, Package_LGA:LGA-14_3x5mm_P0.8mm_LayoutBorder1x6y, F.Cu at (139.0, 106.5)
- moved U3 12.6 mm to (162.0, 128.5)
- moved U1 7.00 mm to (139.0, 75.0)
- moved H2 1.00 mm to (130.0, 57.0)
Connections:
- U2 pad 15: /Alimentacion y cargador/SYSOFF -> GND
Routing:
- net GND: track 1.34 -> 19.0 mm, vias 33 -> 36
- net /Alimentacion y cargador/SYSOFF: track 17.6 -> 0.00 mm, vias 3 -> 0
- removed copper zone on B.Cu, net GND
- removed copper zone on F.Cu, net GND
- removed copper zone on In1.Cu, net GND
Other:
- board size 26 x 109 mm -> 26 x 108 mm

Commit message: Casi que placa lista
Parts:
- added C10: 1uF, Capacitor_SMD:C_0402_1005Metric, F.Cu at (139.0, 132.0)
- added C11: 100nF, Capacitor_SMD:C_0402_1005Metric, F.Cu at (134.2, 132.2)
- added C12: 10uF, TNG_Passives:C_0603, F.Cu at (134.0, 131.0)
- added C13: 100nF, Capacitor_SMD:C_0402_1005Metric, F.Cu at (136.8, 108.0)
- added C14: 100nF, Capacitor_SMD:C_0402_1005Metric, F.Cu at (141.2, 80.2)
- added Q1: AO3401A, Package_TO_SOT_SMD:SOT-23, F.Cu at (132.2, 72.0)
- added R14: 10K, Resistor_SMD:R_0402_1005Metric, F.Cu at (144.8, 118.5)
- added R15: 3K3, Resistor_SMD:R_0402_1005Metric, F.Cu at (143.0, 114.5)
- added R3: 10K, Resistor_SMD:R_0402_1005Metric, F.Cu at (138.0, 132.0)
- added R4: 3K3, Resistor_SMD:R_0402_1005Metric, F.Cu at (141.5, 115.0)
- added R8: 10K, Resistor_SMD:R_0402_1005Metric, F.Cu at (132.5, 75.0)
- added SW1: TS-1088-AR02016, footprints:TS-1088-AR02016, F.Cu at (135.0, 137.0)
- added SW2: TS-1088-AR02016, footprints:TS-1088-AR02016, F.Cu at (135.0, 113.0)
- added TP1: TP, TestPoint:TestPoint_Pad_D1.5mm, F.Cu at (128.5, 97.8)
- added TP2: TP, TestPoint:TestPoint_Pad_D1.5mm, F.Cu at (128.5, 94.3)
- added TP3: TP, TestPoint:TestPoint_Pad_D1.5mm, F.Cu at (128.5, 90.8)
- added TP4: BAT+, TestPoint:TestPoint_Loop_D1.80mm_Drill1.0mm_Beaded, F.Cu at (146.5, 143.5)
- added U7: MAX17048G+T10, Package_DFN_QFN:TDFN-8-1EP_2x2mm_P0.5mm_EP0.8x1.2mm, F.Cu at (140.8, 82.5)
- U5: value ADXL343 -> ADXL345
- moved D1 44.9 mm to (128.5, 149.5)
- moved R18 43.4 mm to (128.5, 146.8)
- moved R16 26.3 mm to (133.6, 147.4)
- moved C9 25.9 mm to (136.8, 104.8), turned to -90 degrees
- moved C7 25.0 mm to (150.0, 104.0), turned to 90 degrees
- moved R17 24.4 mm to (134.6, 147.4)
- moved U3 24.4 mm to (146.8, 109.5)
- moved C6 23.9 mm to (148.5, 104.5)
- moved C5 17.2 mm to (148.5, 114.2), turned to 180 degrees
- moved R11 14.6 mm to (150.2, 141.5), turned to 0 degrees
- moved R10 12.1 mm to (150.8, 138.6), turned to -90 degrees
Connections:
- C9 pad 1: unconnected-(C9-Pad1) -> +3V3
- C9 pad 2: unconnected-(C9-Pad2) -> GND
- D1 pad 1: Net-(D1-K) -> GND
- D1 pad 2: unconnected-(D1-A-Pad2) -> Net-(D1-A)
- J2 pad 1: unconnected-(J2-A-Pad1) -> /SW_MULT_A
- J2 pad 2: unconnected-(J2-B-Pad2) -> /SW_MULT_B
- J2 pad 3: unconnected-(J2-C-Pad3) -> /SW_MULT_C
- J2 pad 4: unconnected-(J2-Com-Pad4) -> GND
- J2 pad 5: unconnected-(J2-D-Pad5) -> /SW_MULT_D
- J2 pad 6: unconnected-(J2-Cen-Pad6) -> /SW_MULT_pul
- J3 pad 1: unconnected-(J3-Pad1) -> /SW_ROT_1
- J3 pad 2: unconnected-(J3-Pad2) -> /SW_ROT_2
- J3 pad C: unconnected-(J3-PadC) -> GND
- J3 pad T: unconnected-(J3-PadT) -> /SW_ROT_T
- R16 pad 1: /USB_D+ -> /USB_D-
- R16 pad 2: /MCU/USB_DP -> /MCU/USB_DN
- R17 pad 1: /USB_D- -> /USB_D+
- R17 pad 2: /MCU/USB_DN -> /MCU/USB_DP
- R18 pad 1: Net-(D1-K) -> /MCU/IO8
- R18 pad 2: GND -> Net-(D1-A)
- U1 pad 2: +3V3 -> Net-(Q1-D)
- U5 pad 1: unconnected-(U5-Vdd_I/O-Pad1) -> +3V3
- U5 pad 12: unconnected-(U5-SDO/ADDR-Pad12) -> GND
- U5 pad 13: unconnected-(U5-SDA/SDI/SDIO-Pad13) -> /MCU/SDA_IMU
- U5 pad 14: unconnected-(U5-SCL/SCLK-Pad14) -> /MCU/SCL_IMU
- U5 pad 2: Net-(U5-GND-Pad2) -> GND
- U5 pad 4: Net-(U5-GND-Pad2) -> GND
- U5 pad 5: Net-(U5-GND-Pad2) -> GND
- U5 pad 6: unconnected-(U5-Vs-Pad6) -> +3V3
- U5 pad 7: unconnected-(U5-~{CS}-Pad7) -> +3V3
- U5 pad 8: unconnected-(U5-INT1-Pad8) -> /MCU/INT
- U6 pad 1: Net-(U6-GND-Pad1) -> GND
- U6 pad 10: unconnected-(U6-IO5-Pad10) -> /SW_ROT_2
- U6 pad 11: Net-(U6-GND-Pad1) -> GND
- U6 pad 12: unconnected-(U6-IO0-Pad12) -> /SW_MULT_A
- U6 pad 13: unconnected-(U6-IO1-Pad13) -> /SW_MULT_C
- U6 pad 14: Net-(U6-GND-Pad1) -> GND
- U6 pad 15: unconnected-(U6-IO6-Pad15) -> /SW_ROT_1
- U6 pad 16: unconnected-(U6-IO7-Pad16) -> /SW_ROT_T
- U6 pad 17: unconnected-(U6-IO12-Pad17) -> /MCU/USB_DN
- U6 pad 18: unconnected-(U6-IO13-Pad18) -> /MCU/USB_DP
- U6 pad 19: unconnected-(U6-IO14-Pad19) -> /SW_MULT_D
- U6 pad 2: Net-(U6-GND-Pad1) -> GND
- U6 pad 20: unconnected-(U6-IO15-Pad20) -> /SW_MULT_pul
- U6 pad 22: unconnected-(U6-IO8-Pad22) -> /MCU/IO8
- U6 pad 23: unconnected-(U6-IO9-Pad23) -> /MCU/IO9
- U6 pad 24: unconnected-(U6-IO18-Pad24) -> /DISP_ON
- U6 pad 25: unconnected-(U6-IO19-Pad25) -> /MCU/SCL_IMU
- U6 pad 26: unconnected-(U6-IO20-Pad26) -> /MCU/SDA_IMU
- U6 pad 27: unconnected-(U6-IO21-Pad27) -> /MCU/INT
- U6 pad 28: unconnected-(U6-IO22-Pad28) -> /SDA
- U6 pad 29: unconnected-(U6-IO23-Pad29) -> /SCL
- U6 pad 3: unconnected-(U6-3V3-Pad3) -> +3V3
- U6 pad 30: unconnected-(U6-RXD0-Pad30) -> /MCU/RX
- U6 pad 31: unconnected-(U6-TXD0-Pad31) -> /MCU/TX
- U6 pad 36: Net-(U6-GND-Pad1) -> GND
- U6 pad 37: Net-(U6-GND-Pad1) -> GND
- U6 pad 38: Net-(U6-GND-Pad1) -> GND
- U6 pad 39: Net-(U6-GND-Pad1) -> GND
- U6 pad 40: Net-(U6-GND-Pad1) -> GND
- U6 pad 41: Net-(U6-GND-Pad1) -> GND
- U6 pad 42: Net-(U6-GND-Pad1) -> GND
- U6 pad 43: Net-(U6-GND-Pad1) -> GND
- U6 pad 44: Net-(U6-GND-Pad1) -> GND
- U6 pad 45: Net-(U6-GND-Pad1) -> GND
- U6 pad 46: Net-(U6-GND-Pad1) -> GND
- U6 pad 47: Net-(U6-GND-Pad1) -> GND
- U6 pad 48: Net-(U6-GND-Pad1) -> GND
- U6 pad 49: Net-(U6-GND-Pad1) -> GND
- U6 pad 5: unconnected-(U6-IO2-Pad5) -> /SW_MULT_B
- U6 pad 50: Net-(U6-GND-Pad1) -> GND
- U6 pad 51: Net-(U6-GND-Pad1) -> GND
- U6 pad 52: Net-(U6-GND-Pad1) -> GND
- U6 pad 53: Net-(U6-GND-Pad1) -> GND
- U6 pad 6: unconnected-(U6-IO3-Pad6) -> /PGOOD
- U6 pad 8: unconnected-(U6-EN-Pad8) -> /MCU/EN
- U6 pad 9: unconnected-(U6-IO4-Pad9) -> /CHG
Routing:
- net /VBAT: track 1.00 -> 78.9 mm
- net /SDA: track 0.00 -> 62.3 mm
- net /SCL: track 0.00 -> 61.4 mm
- net /DISP_ON: track 0.00 -> 53.5 mm, vias 0 -> 2
- net /SW_MULT_A: track 0.00 -> 47.1 mm, vias 0 -> 2
- net /MCU/SCL_IMU: track 0.00 -> 43.0 mm
- net /SW_ROT_1: track 0.00 -> 42.1 mm, vias 0 -> 2
- net /SW_ROT_2: track 0.00 -> 41.2 mm, vias 0 -> 2
- net /SW_MULT_B: track 0.00 -> 40.6 mm, vias 0 -> 2
- net /MCU/IO8: track 0.00 -> 39.8 mm, vias 0 -> 2
- net /CHG: track 0.00 -> 36.2 mm, vias 0 -> 2
- net /MCU/SDA_IMU: track 0.00 -> 35.8 mm, vias 0 -> 2
- net /SW_ROT_T: track 0.00 -> 35.7 mm, vias 0 -> 2
- net /SW_MULT_C: track 0.00 -> 35.5 mm, vias 0 -> 2
- net /SW_MULT_pul: track 0.00 -> 35.0 mm, vias 0 -> 2
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- added copper zone on F.Cu, net +3V3
- added copper zone on In2.Cu, net +3V3
- added copper zone on B.Cu, net GND
- added copper zone on F.Cu, net GND
- added copper zone on In1.Cu, net GND
- added copper zone on In2.Cu, net GND

Commit message: listo para fabricar
Parts:
- added G***: LOGO, LOGO, F.Cu at (142.4, 58.1)
- R16, R17: value 27 -> 22
- moved C10 1.68 mm to (137.5, 103.2), turned to 180 degrees
- renumbered TP4 to B+, C9 to C10, C13 to C11, C10 to C12, C11 to C13, C12 to C14, C14 to C9, Q4 to Q2, R12 to R10, R13 to R11, R4 to R12, R15 to R13, R3 to R15, R8 to R3, R5 to R4, R6 to R5, R7 to R6, R9 to R7, R10 to R8, R11 to R9, SW2 to SW1, SW1 to SW2, TP1 to TP2, TP2 to TP3, TP3 to TP4, U7 to U6, U6 to U7
Routing:
- net /SW_MULT_C: track 35.5 -> 36.9 mm
- net GND: vias 59 -> 61
Other:
- board text added: "B+"
- board text added: "B-"
- board text added: "BOOT"
- board text added: "G"
- board text added: "RST"
- board text added: "RX"
- board text added: "TX"

Commit message: Fabricado
Other:
- board text added: "ESP32-C6 Portatil Rev 1.0"
Changed lines of the file:
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@@
 		)
 		(pad "1" smd roundrect
-			(at -5.1 -3.25)
-			(size 1.4 1.5)
+			(at -5.5 -3.25)
+			(size 1.7 1.5)
 			(layers "F.Cu" "F.Mask" "F.Paste")
 			(roundrect_rratio 0.15)
@@
 		)
 		(pad "2" smd roundrect
-			(at -5.1 0.45)
-			(size 1.4 1.3)
+			(at -5.5 0.45)
+			(size 1.7 1.3)
 			(layers "F.Cu" "F.Mask" "F.Paste")
 			(roundrect_rratio 0.15)
@@
 		)
 		(pad "3" smd roundrect
-			(at -5.1 3.25)
-			(size 1.4 1.5)
+			(at -5.5 3.25)
+			(size 1.7 1.5)
 			(layers "F.Cu" "F.Mask" "F.Paste")
 			(roundrect_rratio 0.15)
@@
 		)
 		(pad "4" smd roundrect
-			(at 5.1 3.25)
-			(size 1.4 1.5)
+			(at 5.5 3.25)
+			(size 1.7 1.5)
 			(layers "F.Cu" "F.Mask" "F.Paste")
 			(roundrect_rratio 0.15)
@@
 		)
 		(pad "5" smd roundrect
-			(at 5.1 0.45)
-			(size 1.4 1.3)
+			(at 5.5 0.45)
+			(size 1.7 1.3)
 			(layers "F.Cu" "F.Mask" "F.Paste")
 			(roundrect_rratio 0.15)
@@
 		)
 		(pad "6" smd roundrect
-			(at 5.1 -3.25)
-			(size 1.4 1.5)
+			(at 5.5 -3.25)
+			(size 1.7 1.5)
 			(layers "F.Cu" "F.Mask" "F.Paste")
 			(roundrect_rratio 0.15)
@@
 		(layer "Edge.Cuts")
 	)
+	(gr_text "ESP32-C6\nPortatil Rev 1.0"
+		(at 149.75 123.25 90)
+		(layer "F.SilkS")
+		(effects
+			(font
+				(size 1 1)
+				(thickness 0.15)
+			)
+		)
+	)
 	(gr_text "BOOT"
 		(at 135 115.5 0)
@@
 	)
 	(segment
-		(start 145.75 95.5)
+		(start 146 95.25)
 		(end 146.25 95)
 		(width 0.2)
@@
 	)
 	(via
-		(at 145.75 95.5)
+		(at 146 95.25)
 		(size 0.5)
 		(drill 0.3)
@@
 	(segment
 		(start 144 97.25)
-		(end 145.75 95.5)
+		(end 144 111)
 		(width 0.2)
 		(layer "B.Cu")
@@
 	)
 	(segment
-		(start 144 111)
-		(end 144 97.25)
+		(start 146.25 113.25)
+		(end 146.25 122.25)
 		(width 0.2)
 		(layer "B.Cu")
@@
 	)
 	(segment
-		(start 143.5 125)
-		(end 146.25 122.25)
+		(start 146 95.25)
+		(end 144 97.25)
 		(width 0.2)
 		(layer "B.Cu")
@@
 	(segment
 		(start 146.25 122.25)
-		(end 146.25 113.25)
+		(end 143.5 125)
 		(width 0.2)
 		(layer "B.Cu")
@@
 	)
 	(segment
-		(start 146.25 113.25)
-		(end 144 111)
+		(start 144 111)
+		(end 146.25 113.25)
 		(width 0.2)
 		(layer "B.Cu")
